Commit message: feat: weigted psuedo inverse for whole body motion

File: src/mobis_description/urdf/mobile_ur5e.urdf (robot description, URDF)
Before this commit: robot mobile_ur5e, 23 links, 22 joints
Joints:
- joint wrist_tool0: type revolute -> fixed

Commit message: bug: lift simulation unfuntional

File: src/mobis_description/urdf/mobile_ur5e.urdf (robot description, URDF)
Before this commit: robot mobile_ur5e, 23 links, 22 joints
Joints:
- joint f_l_prismatic_joint: limit lower=-0.25 upper=0.2 effort=100000 velocity=100 -> lower=-0.25 upper=0.0 effort=100000 velocity=10
- joint f_r_prismatic_joint: limit lower=-0.25 upper=0.2 effort=100000 velocity=100 -> lower=-0.25 upper=0.0 effort=100000 velocity=10
- joint r_l_prismatic_joint: limit lower=-0.25 upper=0.2 effort=100000 velocity=100 -> lower=-0.25 upper=0.0 effort=100000 velocity=10
- joint r_r_prismatic_joint: limit lower=-0.25 upper=0.2 effort=100000 velocity=100 -> lower=-0.25 upper=0.0 effort=100000 velocity=10

Commit message: Add: getmodel

File: src/mobis_description/urdf/mobile_ur5e.urdf (robot description, URDF)
Before this commit: robot mobile_ur5e, 23 links, 22 joints
Links:
- link base_link: mass 10 -> 50
- link base_link_inertia: mass 4.0 -> 4
- link forearm_link: mass 2.275 -> 2.846
- link shoulder_link: mass 3.7 -> 3.761
- link upper_arm_link: mass 8.393 -> 8.058
- link wrist_1_link: mass 1.219 -> 1.37
- link wrist_2_link: mass 1.219 -> 1.3
- link wrist_3_link: mass 0.1879 -> 0.365
Joints:
- joint f_l_prismatic_joint: limit lower=-0.25 upper=0.0 effort=100000 velocity=10 -> lower=-0.25 upper=0.2 effort=100000 velocity=100
- joint f_r_prismatic_joint: limit lower=-0.25 upper=0.0 effort=100000 velocity=10 -> lower=-0.25 upper=0.2 effort=100000 velocity=100
- joint r_l_prismatic_joint: limit lower=-0.25 upper=0.0 effort=100000 velocity=10 -> lower=-0.25 upper=0.2 effort=100000 velocity=100
- joint r_r_prismatic_joint: limit lower=-0.25 upper=0.0 effort=100000 velocity=10 -> lower=-0.25 upper=0.2 effort=100000 velocity=100

File: src/mobis_description/urdf/ur5e.urdf (robot description, URDF)
Before this commit: robot mobile_ur5e, 13 links, 12 joints
Links:
- link base_link_inertia: geometry collision mesh filename=$(find mobis_description)/meshes/ur5e/collision/base.stl; visual mesh filename=$(find mobis_description)/meshes/ur5e/visual/base.dae
- link forearm_link: geometry collision mesh filename=$(find mobis_description)/meshes/ur5e/collision/forearm.stl; visual mesh filename=$(find mobis_description)/meshes/ur5e/visual/forearm.dae
- link shoulder_link: geometry collision mesh filename=$(find mobis_description)/meshes/ur5e/collision/shoulder.stl; visual mesh filename=$(find mobis_description)/meshes/ur5e/visual/shoulder.dae
- link upper_arm_link: geometry collision mesh filename=$(find mobis_description)/meshes/ur5e/collision/upperarm.stl; visual mesh filename=$(find mobis_description)/meshes/ur5e/visual/upperarm.dae
- link wrist_1_link: geometry collision mesh filename=$(find mobis_description)/meshes/ur5e/collision/wrist1.stl; visual mesh filename=$(find mobis_description)/meshes/ur5e/visual/wrist1.dae
- link wrist_2_link: geometry collision mesh filename=$(find mobis_description)/meshes/ur5e/collision/wrist2.stl; visual mesh filename=$(find mobis_description)/meshes/ur5e/visual/wrist2.dae
- link wrist_3_link: geometry collision mesh filename=$(find mobis_description)/meshes/ur5e/collision/wrist3.stl; visual mesh filename=$(find mobis_description)/meshes/ur5e/visual/wrist3.dae

Commit message: Feat task1: whole body impedance control

File: src/mobis_description/urdf/mobile_ur5e.urdf (robot description, URDF)
Before this commit: robot mobile_ur5e, 23 links, 22 joints
Joints:
- joint f_l_prismatic_joint: limit lower=-0.25 upper=0.2 effort=100000 velocity=100 -> lower=-0.25 upper=0.0 effort=100000 velocity=100
- joint f_r_prismatic_joint: limit lower=-0.25 upper=0.2 effort=100000 velocity=100 -> lower=-0.25 upper=0.0 effort=100000 velocity=100
- joint r_l_prismatic_joint: limit lower=-0.25 upper=0.2 effort=100000 velocity=100 -> lower=-0.25 upper=0.0 effort=100000 velocity=100
- joint r_r_prismatic_joint: limit lower=-0.25 upper=0.2 effort=100000 velocity=100 -> lower=-0.25 upper=0.0 effort=100000 velocity=100

Commit message: Add: mobile position estimation

File: src/mobis_description/urdf/mobile_ur5e.urdf (robot description, URDF)
Before this commit: robot mobile_ur5e, 23 links, 22 joints
Links:
- link base_link: mass 50 -> 10
- link f_l_rotate: mass 0.35 -> 1.89
- link r_l_rotate: mass 0.35 -> 1.89
- link r_r_rotate: mass 0.35 -> 1.89
Joints:
- joint f_l_prismatic_joint: limit lower=-0.25 upper=0.0 effort=100000 velocity=100 -> lower=-0.25 upper=0.0 effort=1000000 velocity=10000
- joint f_r_prismatic_joint: limit lower=-0.25 upper=0.0 effort=100000 velocity=100 -> lower=-0.25 upper=0.0 effort=100000 velocity=1000
- joint r_r_prismatic_joint: limit lower=-0.25 upper=0.0 effort=100000 velocity=100 -> lower=-0.25 upper=0.0 effort=100000 velocity=1000
- joint r_r_rotate_joint: limit effort=100 velocity=100 -> effort=100000 velocity=1000
