Commit message: FIX: LPFiltered DOB

File: src/mobis_description/urdf/ur5e_.urdf (robot description, URDF)
Before this commit: robot ur5e_robot, 11 links, 10 joints
Links:
- link forearm_link: mass 2.275 -> 2.846
- link shoulder_link: mass 3.7 -> 3.761
- link upper_arm_link: mass 8.393 -> 8.058
- link wrist_1_link: mass 1.219 -> 1.37
- link wrist_2_link: mass 1.219 -> 1.3
- link wrist_3_link: mass 0.1879 -> 0.365
